File: RevA.sch (EAGLE design)
At the start: 62 parts, among them IC1 MAX31855, IC10 DS3231/SO, IC3 MAX31855, IC4 MAX31855, IC5 MAX31855, IC9 ATMEGA32U4-AU, J1 1X2-3.5MM, J2 1X2-3.5MM, J3 1X2-3.5MM, J4 1X2-3.5MM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

Commit message: Cleaned up the layout
Changed lines of the file:
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@@
 <?xml version="1.0" encoding="utf-8"?>
 <!DOCTYPE eagle SYSTEM "eagle.dtd">
-<eagle version="9.1.0">
+<eagle version="9.1.3">
 <drawing>
 <settings>
@@
 <pinref part="IC1" gate="G$1" pin="T-"/>
 <wire x1="40.64" y1="182.88" x2="48.26" y2="182.88" width="0.1524" layer="91"/>
+<junction x="30.48" y="187.96"/>
 </segment>
 </net>
@@
 <wire x1="248.92" y1="27.94" x2="264.16" y2="27.94" width="0.1524" layer="91"/>
 <label x="248.92" y="27.94" size="1.27" layer="95" rot="R180" xref="yes"/>
+<junction x="264.16" y="27.94"/>
 </segment>
 </net>
@@
 <pinref part="IC3" gate="G$1" pin="T-"/>
 <wire x1="40.64" y1="132.08" x2="48.26" y2="132.08" width="0.1524" layer="91"/>
+<junction x="30.48" y="137.16"/>
 </segment>
 </net>
@@
 <pinref part="IC4" gate="G$1" pin="T-"/>
 <wire x1="38.1" y1="78.74" x2="45.72" y2="78.74" width="0.1524" layer="91"/>
-</segment>
-</net>
+<junction x="27.94" y="83.82"/>
+</segment>
+</net>
